File: rat_board.kicad_pcb (KiCad board)
At the start: 2 copper layers, 2 parts

Commit message: update
Parts:
- removed the REF** at (109.2, 86.4)
- removed the REF** at (101.6, 73.7)
- added J1: Conn_01x02, Connector_JST:JST_XH_B2B-XH-A_1x02_P2.50mm_Vertical, F.Cu at (179.7, 76.5)
- added J2: Conn_01x04, Connector_JST:JST_XH_B4B-XH-A_1x04_P2.50mm_Vertical, F.Cu at (179.7, 124.5)
- added J3: Conn_01x02, Connector_JST:JST_XH_B2B-XH-A_1x02_P2.50mm_Vertical, F.Cu at (179.7, 84.3)
- added J4: Conn_01x02, Connector_JST:JST_XH_B2B-XH-A_1x02_P2.50mm_Vertical, F.Cu at (179.7, 92.1)
- added J5: Conn_01x02, Connector_JST:JST_XH_B2B-XH-A_1x02_P2.50mm_Vertical, F.Cu at (179.7, 99.9)
- added J6: Conn_01x03, Connector_JST:JST_XH_B3B-XH-A_1x03_P2.50mm_Vertical, F.Cu at (179.7, 109.2)
- added R1: 10k, Resistor_THT:R_Axial_DIN0207_L6.3mm_D2.5mm_P7.62mm_Horizontal, F.Cu at (177.8, 116.8)
- added REF**: MountingHole_3.2mm_M3, MountingHole:MountingHole_3.2mm_M3, F.Cu at (195.0, 66.0)
- added REF**: MountingHole_3.2mm_M3, MountingHole:MountingHole_3.2mm_M3, F.Cu at (148.0, 133.0)
- added REF**: MountingHole_3.2mm_M3, MountingHole:MountingHole_3.2mm_M3, F.Cu at (195.0, 133.0)
- added REF**: MountingHole_3.2mm_M3, MountingHole:MountingHole_3.2mm_M3, F.Cu at (148.0, 66.0)
- added U1: ~, mori:ESP32, F.Cu at (161.7, 121.8)
- added U2: DRV8835, mori:DRV8835, F.Cu at (191.2, 77.3)
Routing:
- net Net-(J1-Pin_1): track 0.00 -> 142.5 mm
- net +6V: track 0.00 -> 127.1 mm
- net Net-(J5-Pin_1): track 0.00 -> 55.3 mm
- net SDA: track 0.00 -> 53.3 mm
- net Net-(U1-3V3): track 0.00 -> 53.2 mm
- net Net-(J5-Pin_2): track 0.00 -> 51.0 mm
- net SCL: track 0.00 -> 50.9 mm
- net 3.3V-1: track 0.00 -> 42.4 mm
- net AIN2: track 0.00 -> 41.8 mm
- net MODE: track 0.00 -> 41.7 mm
- net BIN1: track 0.00 -> 40.0 mm
- net AIN1: track 0.00 -> 39.5 mm
- net BIN2: track 0.00 -> 35.0 mm
- net 3.3V-2: track 0.00 -> 24.9 mm
- net Net-(J4-Pin_1): track 0.00 -> 15.8 mm
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- added copper zone on B.Cu, net GND
- added copper zone on F.Cu, net GND
Other:
- board outline added: 53.3 x 72.6 mm
