File: rat_board.kicad_sch (KiCad schematic)
At the start: 1 part

Commit message: update
Parts:
- added J1, J3, J4, J5, J8: Conn_01x02, Connector_JST:JST_XH_B2B-XH-A_1x02_P2.50mm_Vertical, symbol Connector_Generic:Conn_01x02
- added J2: Conn_01x04, Connector_JST:JST_XH_B4B-XH-A_1x04_P2.50mm_Vertical, symbol Connector_Generic:Conn_01x04
- added J6: Conn_01x03, Connector_JST:JST_XH_B3B-XH-A_1x03_P2.50mm_Vertical, symbol Connector_Generic:Conn_01x03
- added J7: Conn_01x02, symbol Connector_Generic:Conn_01x02
- added R1: 10k, Resistor_THT:R_Axial_DIN0207_L6.3mm_D2.5mm_P7.62mm_Horizontal, symbol Device:R
- added SW1: SW_SPDT, mori:switch, symbol Switch:SW_SPDT
- added U2: DRV8835, mori:DRV8835, symbol morilib:DRV8835
Connections:
- net at U1.1 (3V3): now also R1.1
- net at U1.10 (IO26): now also J1.1 (Pin_1), R1.2
- net GND: now reaches U1.14 (GND)
- net GND: now also U1.32 (GND), U1.38 (GND), J1.2 (Pin_2), J2.4 (Pin_4), J4.2 (Pin_2), J7.2 (Pin_2), J8.2 (Pin_2), U2.6 (GND)
- net 3.3V-1: now reaches U1.15 (IO13)
- net 3.3V-1: now also J2.3 (Pin_3)
- net at U1.23 (IO15): now also J8.1 (Pin_1)
- net at U1.24 (IO2): now also J6.3 (Pin_3)
- net at U1.25 (IO0): now also J6.2 (Pin_2)
- net at U1.26 (IO4): now also J6.1 (Pin_1)
- net at U1.28 (IO17): now also J4.1 (Pin_1)
- net 3.3V-2: now reaches U1.29 (IO5)
- net 3.3V-2: now also U2.7 (Vcc)
- net BIN2: now reaches U1.30 (IO18)
- net BIN2: now also U2.12 (BIN2)
- net BIN1: now reaches U1.31 (IO19)
- net BIN1: now also U2.11 (BIN1)
- net AIN2: now reaches U1.33 (IO21)
- net AIN2: now also U2.10 (AIN2)
- net AIN1: now reaches U1.36 (IO22)
- net AIN1: now also U2.9 (AIN1)
- net MODE: now reaches U1.37 (IO23)
- net MODE: now also U2.8 (MODE)
- net SCL: now reaches U1.6 (IO35)
- net SCL: now also J2.1 (Pin_1)
- net SDA: now reaches U1.7 (IO32)
- net SDA: now also J2.2 (Pin_2)
- net VCC: no longer names the net of U1.19 (5V)
- net VCC: now also SW1.2 (B), U2.1 (VM)
- new net: J3.1 (Pin_1), U2.4 (BOUT1)
- new net: J3.2 (Pin_2), U2.5 (BOUT2)
- new net: J5.1 (Pin_1), U2.2 (AOUT1)
- new net: J5.2 (Pin_2), U2.3 (AOUT2)
- new net +6V: J7.1 (Pin_1), SW1.1 (A)
Other:
- note added: "sw"
