File: v1.1/rat_board.kicad_sch (KiCad schematic)
At the start: 20 parts, among them J1 Conn_01x02, J2 Conn_01x04, J3 Conn_01x02, J5 Conn_01x02, J6 Conn_01x03, J7 Conn_01x02, SW1 SW_SPDT, SW2 SW_Push, U2 DRV8835, U3 NJM2845DL-05

Commit message: feat: 基板できた！
Parts:
- added H1, H2, H3, H4: MountingHole_Pad, MountingHole:MountingHole_3.2mm_M3_Pad, symbol Mechanical:MountingHole_Pad
- BZ1: footprint (none) -> mori:PKM22EPP-40
- C1, C2: footprint (none) -> Capacitor_THT:C_Disc_D7.0mm_W2.5mm_P5.00mm
- D1, D2: footprint mori:LED -> LED_THT:LED_D5.0mm
Connections:
- net AIN1: now also U1.33 (IO21); no longer U1.36 (IO22)
- net AIN2: now also U1.31 (IO19); no longer U1.33 (IO21)
- net BIN1: now also U1.30 (IO18); no longer U1.31 (IO19)
- net BIN2: now also U1.29 (IO5); no longer U1.30 (IO18)
- net BUZZER: now also U1.37 (IO23); no longer U1.23 (IO15)
- net GND: now also D1.1 (K), D2.1 (K); no longer R3.1, R4.1
- net LED_A: now also R3.2, U1.12 (IO14); no longer D1.2 (A), U1.7 (IO32)
- net LED_B: now also R4.2, U1.13 (IO12); no longer D2.2 (A), U1.8 (IO33)
- net LIMIT_SW: now also U1.23 (IO15); no longer U1.10 (IO26)
- net MODE: now also U1.36 (IO22); no longer U1.37 (IO23)
- net RGBLED: now also U1.26 (IO4); no longer U1.27 (IO16)
- net SCL: now also U1.28 (IO17); no longer U1.12 (IO14)
- net SDA: now also U1.27 (IO16); no longer U1.13 (IO12)
- net SW: now also U1.11 (IO27); no longer U1.21 (IO7)
- new net: D2.2 (A), R4.1
- new net: D1.2 (A), R3.1
Other:
- note added: "GPIO6~11まで使用不可 GPIO0,2,5,12,15 を使うのは非推奨"
- note added: "IO15はbootと共有"
- moved on the sheet: D1, D2, R3, R4
